File: FrontInterface/PDMRS232CInterface/RS232CInterface.kicad_pcb.kicad_pcb (KiCad board)
At the start: 2 copper layers, 160 x 100.3 mm, 46 parts, among them IC1 ADM3251EARWZ, J1 Screw_Terminal_01x02, J2 DB9_Female, J4 Conn_01x04, Q1 2N7000, Q2 2N7000, U1 MCP2561-E-SN, U2 MCP16301, U3 BluePill_STM32F103C

Commit message: PCB updated
Parts:
- moved D3 32.5 mm to (134.2, 74.4), turned to 270 degrees
- moved U1 31.6 mm to (174.9, 77.0)
- moved C4 31.5 mm to (169.0, 77.0)
- moved L3 29.8 mm to (136.3, 82.0), turned to 180 degrees
- moved C7 25.6 mm to (152.5, 112.3), turned to 0 degrees
- moved C6 22.4 mm to (152.5, 109.8), turned to 0 degrees
- moved D2 21.3 mm to (158.1, 111.1), turned to 0 degrees
- moved D6 21.1 mm to (139.9, 74.4), turned to 270 degrees
- moved R8 20.5 mm to (133.1, 64.6), turned to 90 degrees
- moved R1 19.0 mm to (145.6, 83.9), turned to 0 degrees
- moved C12 17.2 mm to (154.5, 83.2), turned to 270 degrees
- moved F1 16.8 mm to (161.0, 73.2)
- moved C2 15.1 mm to (152.5, 89.5), turned to 180 degrees
- moved R5 14.8 mm to (154.7, 64.3), turned to 90 degrees
- moved R2 14.8 mm to (145.6, 81.3), turned to 0 degrees
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Routing:
- net +5V: track 0.00 -> 179.1 mm, vias 0 -> 1
- net +3V3: track 0.00 -> 109.1 mm
- net Net-(IC1-Pad9): track 0.00 -> 69.3 mm
- net /CANRX_BP: track 0.00 -> 61.4 mm
- net /CANTX_BP: track 0.00 -> 56.3 mm, vias 0 -> 1
- net Net-(IC1-Pad8): track 0.00 -> 55.9 mm
- net Net-(J4-Pad3): track 0.00 -> 50.2 mm
- net Net-(J4-Pad2): track 0.00 -> 45.9 mm
- net Net-(Q1-Pad1): track 0.00 -> 31.9 mm
- net Net-(C9-Pad1): track 0.00 -> 27.1 mm
- net Net-(D1-Pad2): track 0.00 -> 26.2 mm
- net Net-(D2-Pad1): track 0.00 -> 22.6 mm
- net Net-(C11-Pad1): track 0.00 -> 22.0 mm
- net Net-(Q2-Pad1): track 0.00 -> 19.4 mm
- net Net-(BP_Power1-Pad1): track 11.0 -> 27.1 mm
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
Commit message: Zones and routes updated
Parts:
- moved C14 0.57 mm to (167.0, 50.9)
- moved C8 0.36 mm to (174.8, 72.5), turned to 0 degrees
Connections:
- net GNDPWR renamed GNDS
Routing:
- net +24V: track 0.00 -> 46.1 mm, vias 0 -> 2
- net +5V: track 179.1 -> 182.4 mm
- net +3V3: track 109.1 -> 107.7 mm
- net Net-(D4-Pad1): track 5.06 -> 6.13 mm
- net Net-(Q2-Pad1): track 19.4 -> 20.3 mm
- net /PDM/CANH: track 103.5 -> 102.6 mm
- net Net-(IC1-Pad15): track 6.05 -> 6.85 mm
- net Net-(IC1-Pad9): track 69.3 -> 70.0 mm
- net Net-(Q1-Pad1): track 31.9 -> 31.3 mm
- net Net-(C2-Pad2): track 14.3 -> 14.9 mm
- net /CANRX_BP: track 61.4 -> 62.0 mm
- added copper zone on F.Cu, net GNDS
- removed copper zone on B.Cu, net GNDS

Commit message: PCB Rev0
Parts:
- moved D2 3.50 mm to (161.5, 111.3), turned to 180 degrees
- moved D1 3.06 mm to (161.3, 90.7)
Routing:
- net GND: track 0.00 -> 159.1 mm, vias 0 -> 4
- net +5V: track 182.4 -> 214.3 mm, vias 1 -> 3
- net GNDS: track 0.00 -> 12.5 mm
- net Net-(D2-Pad1): track 22.5 -> 16.2 mm
- net Net-(IC1-Pad9): track 70.0 -> 73.7 mm
- net Net-(IC1-Pad8): track 55.6 -> 58.9 mm
- net Net-(D1-Pad2): track 26.2 -> 22.9 mm
- net Net-(C9-Pad1): track 27.2 -> 25.2 mm
- net +3V3: track 107.7 -> 109.1 mm
- net Net-(IC1-Pad15): track 6.85 -> 7.84 mm
- net Net-(J4-Pad3): track 50.2 -> 51.1 mm
- net Net-(J4-Pad2): track 45.9 -> 46.6 mm
- net /CANTX_BP: track 56.8 -> 56.3 mm, vias 1 -> 0
